File: CowTag_v1/power_management.kicad_sch (KiCad schematic)
At the start: 0 parts

Commit message: Actualización completa de esquemáticos CowTag V1 y corrección en main_mcu.kicad_sch
Other:
- company: (none) -> FarmTag - Proyecto AgTech Chile
- title: (none) -> CowTag - Módulo de Gestión Energética
Changed lines of the file:
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@@
 (kicad_sch
-	(version 20250114)
-	(generator "eeschema")
-	(generator_version "9.0")
-	(paper "A4")
+  (version 20250114)
+  (generator "eeschema")
+  (generator_version "9.0")
+  (uuid "power-mgmt-uuid-002")
+  (paper "A4")
+  (title_block
+    (title "CowTag - Módulo de Gestión Energética")
+    (date "2025-06-22")
+    (rev "v1.1")
+    (company "FarmTag - Proyecto AgTech Chile")
+    (comment 1 "Conversión, regulación y protección energética para dispositivo IoT rural")
+    (comment 2 "Basado en batería Li-Ion 18650 + cargador TP4056 + regulador LDO AMS1117")
+    (comment 3 "Incluye entrada solar, salida 3V3 estabilizada y estado de carga")
+    (comment 4 "Optimizado para zonas rurales sin red eléctrica, enfoque en autonomía")
+  )
+  (symbol_instances
+    (path "/U1" (reference "U1") (value "TP4056_Module") (footprint "Module:TP4056_Protection"))
+    (path "/U2" (reference "U2") (value "AMS1117-3.3") (footprint "Regulator_Linear:AMS1117-3.3_SOT-223"))
+    (path "/BT1" (reference "BT1") (value "Battery_Cell_18650") (footprint "Battery:Battery_Holder_Keystone_18650"))
+    (path "/J1" (reference "J1") (value "Connector_Solar_IN") (footprint "Connector:TerminalBlock_2Pin"))
+    (path "/R1" (reference "R1") (value "R_10k_BAT_STAT") (footprint "Resistor_SMD:R_0603"))
+    (path "/LED1" (reference "LED1") (value "LED_BAT_STATUS") (footprint "LED_SMD:LED_0603"))
+    (path "/C1" (reference "C1") (value "Cout_10uF") (footprint "Capacitor_SMD:C_0603"))
+    (path "/C2" (reference "C2") (value "Cin_10uF") (footprint "Capacitor_SMD:C_0603"))
+    (path "/D1" (reference "D1") (value "TVS_PROTECT") (footprint "Diode_SMD:D_SOD-323"))
+    (path "/F1" (reference "F1") (value "Polyfuse_500mA") (footprint "Fuse:Fuse_0603_1608Metric"))
+  )
 )
